Commit message: add ros2 controller

File: bumperbot_description/urdf/bumperbot_gazebo.xacro (robot description, xacro)
@@ -23,5 +23,5 @@
         <mu2>0.1</mu2>
         <kp>1000000.0</kp>
-        <kd>100</kd>
+        <kd>100.0</kd>
         <minDepth>0.001</minDepth>
         <maxVel>0.1</maxVel>
@@ -31,5 +31,5 @@
         <mu2>0.1</mu2>
         <kp>1000000.0</kp>
-        <kd>100</kd>
+        <kd>100.0</kd>
         <minDepth>0.001</minDepth>
         <maxVel>0.1</maxVel>
@@ -38,10 +38,10 @@
         <xacro:if value="$(arg is_ignition)">
             <plugin filename="ign_ros2_control-system" name="ign_ros2_control::IgnitionROS2ControlPlugin">
-                <parameters></parameters>
+                <parameters>$(find bumperbot_controller)/config/bumperbot_controllers.yaml</parameters>
             </plugin>
         </xacro:if>
         <xacro:unless value="$(arg is_ignition)">
             <plugin filename="gz_ros2_control-system" name="gz_ros2_control::GazeboSimROS2ControlPlugin">
-                <parameters></parameters>
+                <parameters>$(find bumperbot_controller)/config/bumperbot_controllers.yaml</parameters>
             </plugin>
         </xacro:unless>

File: bumperbot_description/urdf/bumperbot_ros2_control.xacro (robot description, xacro)
@@ -20,5 +20,5 @@
             <state_interface name="velocity"/>
         </joint>
-        <joint name="wheel_left_join">
+        <joint name="wheel_left_joint">
             <command_interface name="velocity">
                 <param name="min">-1</param>

Commit message: add imu to urdf

File: bumperbot_description/urdf/bumperbot_gazebo.xacro (robot description, xacro)
@@ -40,4 +40,6 @@
                 <parameters>$(find bumperbot_controller)/config/bumperbot_controllers.yaml</parameters>
             </plugin>
+            <plugin filename="ignition-gazebo-imu-system" name="ignition::gazebo::systems::Imu">
+            </plugin>
         </xacro:if>
         <xacro:unless value="$(arg is_ignition)">
@@ -45,5 +47,57 @@
                 <parameters>$(find bumperbot_controller)/config/bumperbot_controllers.yaml</parameters>
             </plugin>
+            <plugin filename="gz-sim-imu-system" name="gz::sim::systems::Imu">
+            </plugin>
         </xacro:unless>
     </gazebo>
+    <gazebo reference="imu_link">
+        <sensor name="imu" type="imu">
+            <always_on>true</always_on>
+            <update_rate>100.0</update_rate>
+            <gz_frame_id>imu_link</gz_frame_id>
+            <topic>imu</topic>
+            <imu>
+                <angular_velocity>
+                    <x>
+                        <noise type="gaussian">
+                            <mean>0.0</mean>
+                            <stddev>2e-4</stddev>
+                        </noise>
+                    </x>
+                    <y>
+                        <noise type="gaussian">
+                            <mean>0.0</mean>
+                            <stddev>2e-4</stddev>
+                        </noise>
+                    </y>
+                    <z>
+                        <noise type="gaussian">
+                            <mean>0.0</mean>
+                            <stddev>2e-4</stddev>
+                        </noise>
+                    </z>
+                </angular_velocity>
+                <linear_velocity>
+                    <x>
+                        <noise type="gaussian">
+                            <mean>0.0</mean>
+                            <stddev>1.7e-2</stddev>
+                        </noise>
+                    </x>
+                    <y>
+                        <noise type="gaussian">
+                            <mean>0.0</mean>
+                            <stddev>1.7e-2</stddev>
+                        </noise>
+                    </y>
+                    <z>
+                        <noise type="gaussian">
+                            <mean>0.0</mean>
+                            <stddev>1.7e-2</stddev>
+                        </noise>
+                    </z>
+                </linear_velocity>
+            </imu>
+        </sensor>
+    </gazebo>
 </robot>

File: bumperbot_description/urdf/bumperbot_urdf.xacro (robot description, xacro)
@@ -136,3 +136,30 @@
         <origin xyz="-0.047 0 -0.027" rpy="0 0 0"/>
     </joint>
+    <link name="imu_link">
+        <inertial>
+            <origin xyz="-0.00552433659106688 0.000168210391520346 0.000514000497342681" rpy="0 0 0" />
+            <mass value="0.000528415362211671" />
+            <inertia ixx="1.46176048428261E-08" ixy="1.40015117949421E-10" ixz="-1.99633872937403E-12"
+                     iyy="8.59662482954888E-09" iyz="7.52375112767959E-12"
+                     izz="2.30279421279312E-08" />
+        </inertial>
+        <visual>
+            <origin xyz="0 0 0" rpy="0 0 0"/>
+            <geometry>
+                <mesh filename="package://bumperbot_description/meshes/imu_link.STL"/>
+            </geometry>
+        </visual>
+        <visual>
+            <origin xyz="0 0 0" rpy="0 0 0"/>
+            <geometry>
+                <mesh filename="package://bumperbot_description/meshes/imu_link.STL"/>
+            </geometry>
+        </visual>
+    </link>
+    <joint name="imu_joint" type="fixed">
+        <parent link="base_link"/>
+        <child link="imu_link"/>
+        <origin xyz="0 0 0.07" rpy="3.14 0 0"/>
+        <axis xyz="0 0 0"/>
+    </joint>
 </robot>
