Commit message: prepare ros2_control

File: bumperbot_description/urdf/bumperbot_urdf.xacro (robot description, xacro)
@@ -1,6 +1,16 @@
 <?xml version='1.0'?>
 <robot xmlns:xacro="http://www.ros.org/wiki/xacro" name="bumperbot">
+    <xacro:arg name="is_ignition" default="true" />
+    <xacro:include filename="$(find bumperbot_description)/urdf/bumperbot_gazebo.xacro"/>
+    <xacro:include filename="$(find bumperbot_description)/urdf/bumperbot_ros2_control.xacro"/>
     <link name="base_footprint"/>
     <link name="base_link">
+        <inertial>
+            <origin xyz="0 0 0.04" rpy="0.0 0.25 0.3" />
+            <mass value="8.2573504e-01"/>
+            <inertia ixx="2.2124416e-02" ixy="-1.2294101e-04" ixz="3.4938785e-04"
+                    iyy="2.1193702e-02" iyz="-5.0120904e-05"
+                    izz="2.0064271e-02" />
+        </inertial>
         <visual>
             <origin rpy="0 0 0" xyz="0 0 0"/>
@@ -9,4 +19,9 @@
             </geometry>
         </visual>
+        <collision>
+            <geometry>
+                <mesh filename="package://bumperbot_description/meshes/base_link.STL"/>
+            </geometry>
+        </collision>
     </link>
     <joint name="base_joint" type="fixed">
@@ -16,4 +31,11 @@
     </joint>
     <link name="wheel_right_link">
+        <inertial>
+            <origin xyz="0 -0.014 0" rpy="0 0 0" />
+            <mass value="0.0530086090966721" />
+            <inertia ixx="1.88176298336665E-05" ixy="-4.8444933029987E-10" ixz="1.88163708851143E-08"
+                     iyy="3.11510738647764E-05" iyz="-6.93560663069607E-11"
+                     izz="1.8801969558182E-05" />
+        </inertial>
         <visual>
             <origin rpy="${pi/2} 0 0" xyz="0 0 0"/>
@@ -22,4 +44,10 @@
             </geometry>
         </visual>
+        <collision>
+            <origin xyz="0 -0.015 0" rpy="1.57 0 0"/>
+            <geometry>
+                <sphere radius="0.033"/>
+            </geometry>
+        </collision>
     </link>
     <joint name="wheel_right_joint" type="continuous">
@@ -30,4 +58,11 @@
     </joint>
     <link name="wheel_left_link">
+        <inertial>
+            <origin xyz="0 0.014 0" rpy="0 0 0" />
+            <mass value="0.0530086043217644" />
+            <inertia ixx="1.8792911368909E-05"  ixy="3.31256392204584E-10" ixz="-1.14082001662767E-08"
+                     iyy="3.11510738759073E-05" iyz="-3.60499245082192E-10"
+                     izz="1.88266886146847E-05" />
+        </inertial>
         <visual>
             <origin xyz="0 0 0" rpy="${-pi/2} 0 0"/>
@@ -36,4 +71,10 @@
             </geometry>
         </visual>
+        <collision>
+            <origin xyz="0 0.015 0" rpy="1.57 0 0"/>
+            <geometry>
+                <sphere radius="0.033"/>
+            </geometry>
+        </collision>
     </link>
     <joint name="wheel_left_joint" type="continuous">
@@ -44,4 +85,11 @@
     </joint>
     <link name="caster_front_link">
+        <inertial>
+            <origin xyz="3.89968128948481E-07 2.40073004698083E-07 0.00219173397061506" rpy="0 0 0" />
+            <mass value="1.44379265037903E-06" />
+            <inertia ixx="7.23075276010246E-11" ixy="-6.10956883467859E-16" ixz="2.22849693525031E-15"
+                     iyy="3.8713793085917E-11"  iyz="2.93909858781952E-15"
+                     izz="1.00967486676306E-10" />
+        </inertial>
         <visual>
             <origin xyz="0 0 0" rpy="0 0 0"/>
@@ -50,4 +98,10 @@
             </geometry>
         </visual>
+        <collision>
+            <origin xyz="0 0 0" rpy="0 0 0"/>
+            <geometry>
+                <sphere radius="0.005"/>
+            </geometry>
+        </collision>
     </link>
     <joint name="caster_front_joint" type="fixed">
@@ -57,4 +111,11 @@
     </joint>
     <link name="caster_rear_link">
+        <inertial>
+            <origin xyz="3.8996812895542E-07 2.40073004698083E-07 0.00219173397061509" rpy="0 0 0" />
+            <mass value="1.44379265037902E-06" />
+            <inertia ixx="7.23075276010246E-11" ixy="-6.10956872363424E-16" ixz="2.22849693527207E-15"
+                     iyy="3.87137930859167E-11" iyz="2.939098587861E-15"
+                     izz="1.00967486676306E-10" />
+        </inertial>
         <visual>
             <origin xyz="0 0 0" rpy="0 0 0"/>
@@ -63,4 +124,10 @@
             </geometry>
         </visual>
+        <collision>
+            <origin xyz="0 0 0" rpy="0 0 0"/>
+            <geometry>
+                <sphere radius="0.005"/>
+            </geometry>
+        </collision>
     </link>
     <joint name="caster_rear_joint" type="fixed">

Commit message: sensor fusion with kalman ifter

File: bumperbot_description/urdf/bumperbot_urdf.xacro (robot description, xacro)
@@ -160,5 +160,5 @@
         <parent link="base_link"/>
         <child link="imu_link"/>
-        <origin xyz="0 0 0.07" rpy="3.14 0 0"/>
+        <origin xyz="0 0 0.07" rpy="0 0 0"/>
         <axis xyz="0 0 0"/>
     </joint>

Commit message: add gazebo world arg to launch file

File: bumperbot_description/urdf/bumperbot_urdf.xacro (robot description, xacro)
@@ -18,4 +18,5 @@
                 <mesh filename="package://bumperbot_description/meshes/base_link.STL"/>
             </geometry>
+            <material name="black"/>
         </visual>
         <collision>
@@ -43,4 +44,5 @@
                 <mesh filename="package://bumperbot_description/meshes/wheel_right_link.STL"/>
             </geometry>
+            <material name="blue"/>
         </visual>
         <collision>
@@ -70,4 +72,5 @@
                 <mesh filename="package://bumperbot_description/meshes/wheel_left_link.STL"/>
             </geometry>
+            <material name="blue"/>
         </visual>
         <collision>
@@ -97,4 +100,5 @@
                 <mesh filename="package://bumperbot_description/meshes/caster_front_link.STL"/>
             </geometry>
+            <material name="silver"/>
         </visual>
         <collision>
@@ -123,4 +127,5 @@
                 <mesh filename="package://bumperbot_description/meshes/caster_rear_link.STL"/>
             </geometry>
+            <material name="silver"/>
         </visual>
         <collision>
@@ -149,4 +154,5 @@
                 <mesh filename="package://bumperbot_description/meshes/imu_link.STL"/>
             </geometry>
+            <material name="blue"/>
         </visual>
         <visual>
@@ -163,3 +169,12 @@
         <axis xyz="0 0 0"/>
     </joint>
+    <material name="blue">
+        <color rgba="0 0 1 1"/>
+    </material>
+    <material name="black">
+        <color rgba="0 0 0 1"/>
+    </material>
+    <material name="silver">
+        <color rgba="0.79 0.82 0.93 1"/>
+    </material>
 </robot>

Commit message: add node that calculate rotation and translation of the robot

File: bumperbot_description/urdf/bumperbot_urdf.xacro (robot description, xacro)
@@ -145,6 +145,5 @@
             <origin xyz="-0.00552433659106688 0.000168210391520346 0.000514000497342681" rpy="0 0 0" />
             <mass value="0.000528415362211671" />
-            <inertia ixx="1.46176048428261E-08" ixy="1.40015117949421E-10" ixz="-1.99633872937403E-12"
-                     iyy="8.59662482954888E-09" iyz="7.52375112767959E-12"
+            <inertia ixx="1.4618.62482954888E-09" iyz="7.52375112767959E-12"
                      izz="2.30279421279312E-08" />
         </inertial>

Commit message: add a lidar to the robot and fix imu inertial

File: bumperbot_description/urdf/bumperbot_urdf.xacro (robot description, xacro)
@@ -145,6 +145,7 @@
             <origin xyz="-0.00552433659106688 0.000168210391520346 0.000514000497342681" rpy="0 0 0" />
             <mass value="0.000528415362211671" />
-            <inertia ixx="1.4618.62482954888E-09" iyz="7.52375112767959E-12"
-                     izz="2.30279421279312E-08" />
+            <inertia ixx="1.46176048428261E-08" ixy="1.40015117949421E-10" ixz="-1.99633872937403E-12"
+                    iyy="8.59662482954888E-09" iyz="7.52375112767959E-12"
+                    izz="2.30279421279312E-08" />
         </inertial>
         <visual>
@@ -167,4 +168,31 @@
         <origin xyz="0 0 0.07" rpy="0 0 0"/>
         <axis xyz="0 0 0"/>
+    </joint>
+    <link name="laser_link">
+        <inertial>
+            <origin xyz="-0.011945780406062 -0.000381929217680526 -0.0170649378129477" rpy="0 0 0" />
+            <mass value="0.073084435549317" />
+            <inertia ixx="1.96074931730795E-05" ixy="-3.62091076640009E-07" ixz="4.28230084046735E-07"
+                     iyy="2.40983835136327E-05" iyz="1.50180909250652E-08"
+                     izz="4.14184164228595E-05" />
+        </inertial>
+        <visual>
+            <origin xyz="0 0 0" rpy="0 0 0"/>
+            <geometry>
+                <mesh filename="package://bumperbot_description/meshes/laser_link.STL"/>
+            </geometry>
+            <material name="black"/>
+        </visual>
+        <collision>
+            <origin xyz="0 0 0" rpy="0 0 0"/>
+            <geometry>
+                <mesh filename="package://bumperbot_description/meshes/laser_link.STL"/>
+            </geometry>
+        </collision>
+    </link>
+    <joint name="laser_joint" type="fixed">
+        <parent link="base_link"/>
+        <child link="laser_link"/>
+        <origin xyz="0 0 0.1208" rpy="0 0 3.14"/>
     </joint>
     <material name="blue">

Commit message: fix robot unbalance

File: bumperbot_description/urdf/bumperbot_urdf.xacro (robot description, xacro)
@@ -33,58 +33,59 @@
     <link name="wheel_right_link">
         <inertial>
-            <origin xyz="0 -0.014 0" rpy="0 0 0" />
-            <mass value="0.0530086090966721" />
-            <inertia ixx="1.88176298336665E-05" ixy="-4.8444933029987E-10" ixz="1.88163708851143E-08"
-                     iyy="3.11510738647764E-05" iyz="-6.93560663069607E-11"
-                     izz="1.8801969558182E-05" />
-        </inertial>
-        <visual>
-            <origin rpy="${pi/2} 0 0" xyz="0 0 0"/>
-            <geometry>
-                <mesh filename="package://bumperbot_description/meshes/wheel_right_link.STL"/>
-            </geometry>
-            <material name="blue"/>
-        </visual>
-        <collision>
-            <origin xyz="0 -0.015 0" rpy="1.57 0 0"/>
-            <geometry>
-                <sphere radius="0.033"/>
-            </geometry>
-        </collision>
-    </link>
-    <joint name="wheel_right_joint" type="continuous">
-        <parent link="base_link"/>
-        <child link="wheel_right_link"/>
-        <origin rpy="0 0 0" xyz="0 -0.07 0"/>
-        <axis xyz="0 1 0"/>
-    </joint>
-    <link name="wheel_left_link">
-        <inertial>
-            <origin xyz="0 0.014 0" rpy="0 0 0" />
-            <mass value="0.0530086043217644" />
-            <inertia ixx="1.8792911368909E-05"  ixy="3.31256392204584E-10" ixz="-1.14082001662767E-08"
-                     iyy="3.11510738759073E-05" iyz="-3.60499245082192E-10"
-                     izz="1.88266886146847E-05" />
-        </inertial>
-        <visual>
-            <origin xyz="0 0 0" rpy="${-pi/2} 0 0"/>
-            <geometry>
-                <mesh filename="package://bumperbot_description/meshes/wheel_left_link.STL"/>
-            </geometry>
-            <material name="blue"/>
-        </visual>
-        <collision>
-            <origin xyz="0 0.015 0" rpy="1.57 0 0"/>
-            <geometry>
-                <sphere radius="0.033"/>
-            </geometry>
-        </collision>
-    </link>
-    <joint name="wheel_left_joint" type="continuous">
-        <parent link="base_link"/>
-        <child link="wheel_left_link"/>
-        <origin xyz="0 0.07 0" rpy="0 0 0"/>
-        <axis xyz="0 1 0"/>
-    </joint>
+          <origin xyz="0 -0.014 0" rpy="0 0 0" />
+          <mass value="0.0530086090966721" />
+          <inertia ixx="1.88176298336665E-05" ixy="-4.8444933029987E-10" ixz="1.88163708851143E-08"
+                   iyy="3.11510738647764E-05" iyz="-6.93560663069607E-11"
+                   izz="1.8801969558182E-05" />
+        </inertial>
+        <visual>
+          <origin xyz="0 0 0" rpy="1.57 0 0" />
+          <geometry>
+            <mesh filename="package://bumperbot_description/meshes/wheel_right_link.STL" />
+          </geometry>
+          <material name="blue"/>
+        </visual>
+        <collision>
+          <origin xyz="0 -0.015 0" rpy="1.57 0 0" />
+          <geometry>
+            <sphere radius="0.033"/>
+          </geometry>
+        </collision>
+      </link>
+      <joint name="wheel_right_joint" type="continuous">
+        <origin xyz="0 -0.0701101849418637 0" rpy="0 0 0" />
+        <parent link="base_link" />
+        <child link="wheel_right_link" />
+        <axis xyz="0 1 0" />
+      </joint>
+      <link
+        name="wheel_left_link">
+        <inertial>
+          <origin xyz="0 0.014 0" rpy="0 0 0" />
+          <mass value="0.0530086043217644" />
+          <inertia ixx="1.8792911368909E-05"  ixy="3.31256392204584E-10" ixz="-1.14082001662767E-08"
+                   iyy="3.11510738759073E-05" iyz="-3.60499245082192E-10"
+                   izz="1.88266886146847E-05" />
+        </inertial>
+        <visual>
+          <origin xyz="0 0 0" rpy="-1.57 0 0" />
+          <geometry>
+            <mesh filename="package://bumperbot_description/meshes/wheel_left_link.STL" />
+          </geometry>
+          <material name="blue"/>
+        </visual>
+        <collision>
+          <origin xyz="0 0.015 0" rpy="-1.57 0 0" />
+          <geometry>
+            <sphere radius="0.033"/>
+          </geometry>
+        </collision>
+      </link>
+      <joint name="wheel_left_joint" type="continuous">
+        <origin xyz="0 0.0701101849418642 0" rpy="0 0 0" />
+        <parent link="base_link" />
+        <child link="wheel_left_link" />
+        <axis xyz="0 1 0" />
+      </joint>
     <link name="caster_front_link">
         <inertial>
@@ -112,5 +113,5 @@
         <parent link="base_link"/>
         <child link="caster_front_link"/>
-        <origin xyz="0.047 0 -0.027" rpy="0 0 0"/>
+        <origin xyz="0.04755 0 -0.028" rpy="0 0 0"/>
     </joint>
     <link name="caster_rear_link">
@@ -139,5 +140,5 @@
         <parent link="base_link"/>
         <child link="caster_rear_link"/>
-        <origin xyz="-0.047 0 -0.027" rpy="0 0 0"/>
+        <origin xyz="-0.047 0 -0.028" rpy="0 0 0"/>
     </joint>
     <link name="imu_link">
